Commit message: Camera Added

File: install/arduinobot_description/share/arduinobot_description/urdf/arduinobot.urdf.xacro (robot description, xacro)
@@ -121,3 +121,17 @@
         <limit lower="0.0" upper="${PI/2}" effort="${effort}" velocity="${velocity}"/>
     </joint>
+<!-- Camera -->
+    <link name="rgb_camera">
+        <visual>
+            <origin rpy="-1.57 0 -1.57" xyz="-0.1 0.125 0.15"/>
+            <geometry>
+                <mesh filename="package://arduinobot_description/meshes/pi_camera.STL" scale="0.01 0.01 0.01"/>
+            </geometry>
+        </visual>
+    </link>
+    <joint name ="rgb_camera_joint" type="fixed">
+        <parent link="base_link"/>
+        <child link = "rgb_camera"/>
+        <origin xyz="0 0.45 0.2" rpy="0 -0.5 1.57"/>
+    </joint>
 </robot>

Commit message: Gazebo simulation added

File: install/arduinobot_description/share/arduinobot_description/urdf/arduinobot.urdf.xacro (robot description, xacro)
@@ -5,5 +5,16 @@
     <xacro:property  name = "velocity" value= "10.0"/>
     <link name = "world"/>
+    <!-- Useful Macros -->
+    <xacro:macro name="default_inertial" params="mass">
+        <inertial>
+            <mass value="${mass}" />
+            <inertia ixx="1.0" ixy="0.0" ixz="0.0"
+                     iyy="1.0" iyz="0.0"
+                     izz="1.0" />
+        </inertial>
+    </xacro:macro>
+    <!-- base_link -->
     <link name = "base_link">
+        <xacro:default_inertial mass="1.0"/>
         <visual>
             <origin rpy="0 0 0" xyz="-0.5 -0.5 0"/>
@@ -12,4 +23,10 @@
             </geometry>
         </visual>
+        <collision>
+            <origin rpy="0 0 0" xyz="-0.5 -0.5 0"/>
+            <geometry>
+                <mesh filename= "package://arduinobot_description/meshes/basement.STL" scale = "0.01 0.01 0.01"/>
+            </geometry>
+        </collision>
     </link>
     <joint name = "virtual_joint" type = "fixed">
@@ -18,5 +35,7 @@
         <origin rpy = "0 0 0" xyz="0 0 0"/>
     </joint>
+    <!-- base_plate -->
     <link name = "base_plate">
+        <xacro:default_inertial mass="0.1"/>
         <visual>
             <origin rpy="0 0 0" xyz="-0.39 -0.39 -0.56"/>
@@ -25,4 +44,10 @@
             </geometry>
         </visual>
+        <collision>
+            <origin rpy="0 0 0" xyz="-0.39 -0.39 -0.56"/>
+            <geometry>
+                <mesh filename= "package://arduinobot_description/meshes/base_plate.STL" scale = "0.01 0.01 0.01"/>
+            </geometry>
+        </collision>
     </link>
     <joint name = "joint_1" type = "revolute">
@@ -35,4 +60,5 @@
     <!-- forward_drive_arm -->
     <link name = "forward_drive_arm">
+        <xacro:default_inertial mass="0.1"/>
         <visual>
             <origin rpy="0 -${PI/2} ${PI/2}" xyz="0.19 0.06 -0.08"/>
@@ -41,4 +67,10 @@
             </geometry>
         </visual>
+        <collision>
+            <origin rpy="0 -${PI/2} ${PI/2}" xyz="0.19 0.06 -0.08"/>
+            <geometry>
+                <mesh filename= "package://arduinobot_description/meshes/forward_drive_arm.STL" scale = "0.01 0.01 0.01"/>
+            </geometry>
+        </collision>
     </link>
     <joint name = "joint_2" type = "revolute">
@@ -51,4 +83,5 @@
     <!-- horizontal_arm -->
     <link name = "horizontal_arm">
+        <xacro:default_inertial mass="0.1"/>
         <visual>
             <origin rpy="${PI/2} 0 ${PI/2}" xyz="-0.03 -0.4 -0.06"/>
@@ -57,4 +90,10 @@
             </geometry>
         </visual>
+        <collision>
+            <origin rpy="${PI/2} 0 ${PI/2}" xyz="-0.03 -0.4 -0.06"/>
+            <geometry>
+                <mesh filename= "package://arduinobot_description/meshes/horizontal_arm.STL" scale = "0.01 0.01 0.01"/>
+            </geometry>
+        </collision>
     </link>
     <joint name = "joint_3" type = "revolute">
@@ -70,4 +109,5 @@
     <!-- claw_support -->
     <link name = "claw_support">
+        <xacro:default_inertial mass="0.05"/>
         <visual>
             <origin rpy="0 0 ${PI/2}" xyz="0 -0.05 -0.15"/>
@@ -76,4 +116,10 @@
             </geometry>
         </visual>
+        <colision>
+            <origin rpy="0 0 ${PI/2}" xyz="0 -0.05 -0.15"/>
+            <geometry>
+                <mesh filename= "package://arduinobot_description/meshes/claw_support.STL" scale = "0.01 0.01 0.01"/>
+            </geometry>
+        </colision>
     </link>
     <joint name = "horizontal_arm_to_claw_support" type = "fixed">
@@ -85,4 +131,5 @@
     <!-- gripper left and right which are the child of claw support -->
     <link name = "gripper_right">
+        <xacro:default_inertial mass="0.01"/>
         <visual>
             <origin rpy="0 0 -${PI/2}" xyz="-0.1 0.5 -0.1"/>
@@ -91,6 +138,13 @@
             </geometry>
         </visual>
+        <collision>
+            <origin rpy="0 0 -${PI/2}" xyz="-0.1 0.5 -0.1"/>
+            <geometry>
+                <mesh filename= "package://arduinobot_description/meshes/right_finger.STL" scale = "0.01 0.01 0.01"/>
+            </geometry>
+        </collision>
     </link>
         <link name = "gripper_left">
+        <xacro:default_inertial mass="0.01"/>
         <visual>
             <origin rpy="0 0 -${PI/2}" xyz="-0.04 0.5 -0.1"/>
@@ -99,4 +153,10 @@
             </geometry>
         </visual>
+        <collision>
+            <origin rpy="0 0 -${PI/2}" xyz="-0.04 0.5 -0.1"/>
+            <geometry>
+                <mesh filename= "package://arduinobot_description/meshes/left_finger.STL" scale = "0.01 0.01 0.01"/>
+            </geometry>
+        </collision>
     </link>
     <joint name = "joint_4" type = "revolute">
@@ -110,5 +170,5 @@
         <limit lower="-${PI/2}" upper="0.0" effort="${effort}" velocity="${velocity}"/>
     </joint>
-        <joint name = "joint_5" type = "revolute">
+    <joint name = "joint_5" type = "revolute">
         <parent link = "claw_support"/>
         <child link = "gripper_left"/>
@@ -121,6 +181,7 @@
         <limit lower="0.0" upper="${PI/2}" effort="${effort}" velocity="${velocity}"/>
     </joint>
-<!-- Camera -->
+<!-- rgb_camera -->
     <link name="rgb_camera">
+        <xacro:default_inertial mass="0.001"/>
         <visual>
             <origin rpy="-1.57 0 -1.57" xyz="-0.1 0.125 0.15"/>
@@ -129,4 +190,10 @@
             </geometry>
         </visual>
+        <collision>
+            <origin rpy="-1.57 0 -1.57" xyz="-0.1 0.125 0.15"/>
+            <geometry>
+                <mesh filename="package://arduinobot_description/meshes/pi_camera.STL" scale="0.01 0.01 0.01"/>
+            </geometry>
+        </collision>
     </link>
     <joint name ="rgb_camera_joint" type="fixed">
